File: power.kicad_sch (KiCad schematic)
At the start: 1 part, among them U2 102110419

Commit message: Add files via upload
Parts:
- removed U2: 102110419, 102110419_SEE, symbol 2025-11-04_02-54-44:102110419
- added U1: ~, symbol Jetson Orin Nano Symbol:4G_Adaptor_and_Antenna
- added U3: ~, symbol Jetson Orin Nano Symbol:R12_Air_Unit
- added jn1: ~, symbol Jetson Orin Nano Symbol:JetsonOrinNano
- added lora_1w1: ~, symbol sky-4:Lora_1W
- added pixhawk1: ~, symbol sky4-sym v2:Pixhawk
- added pm1: ~, symbol sky4-sym:PM07
Connections:
- new net: U1. (USB_IN/OUT), jn1. (USB-C)
- new net: pixhawk1. (I/O_PWM_OUT), pm1. (GND)
- new net: jn1.10 (GPIO15), jn1.8 (GPIO14), jn1.9 (Ground), pixhawk1. (I/O_PWM_OUT)
- new net: U3. (2.4_ANT), pixhawk1. (I/O_PWM_OUT) (x2)
- new net: lora_1w1. (GND), pixhawk1. (I/O_PWM_OUT)
Other:
- note removed: "NVIDIA Jetson Nano"
